Commit message: add inertial values to links

File: description/robot_core.xacro (robot description, xacro)
@@ -17,5 +17,5 @@
      <!-- CHASSIS -->
       <link name="chassis_link" >
-           <visual>
+            <visual>
                 <origin xyz="0.15 0 0.075" rpy="0 0 0" />
                 <geometry>
@@ -23,5 +23,14 @@
                 </geometry>
                 <material name="white" />
-           </visual>
+            </visual>
+            <collision>
+                <origin xyz="0.15 0 0.075" rpy="0 0 0" />
+                <geometry>
+                    <box size="0.3 0.3 0.15" />
+                </geometry>
+            </collision>
+            <xacro:inertial_box mass="0.5" x="0.3" y="0.3" z="0.15">
+                <origin xyz="0.15 0 0.075" rpy="0 0 0"/>
+            </xacro:inertial_box>
       </link>
        <joint name="chassis_joint" type="fixed">
@@ -38,4 +47,13 @@
                 <material name="blue" />
             </visual>
+            <collision>
+                <origin xyz="0.15 0 0.075" rpy="0 0 0" />
+                <geometry>
+                    <box size="0.3 0.3 0.15" />
+                </geometry>
+            </collision>
+            <xacro:inertial_cylinder mass="0.1" length="0.05" radius="0.05">
+                <origin xyz="0 0 0" rpy="0 0 0"/>
+            </xacro:inertial_cylinder>
         </link>
         <joint name="left_wheel_joint" type="continuous">
@@ -59,4 +77,7 @@
                 <material name="blue"/>
             </visual>
+            <xacro:inertial_sphere mass="0.1" radius="0.05">
+                <origin xyz="0 0 0" rpy="0 0 0"/>
+            </xacro:inertial_sphere>
         </link>
         <!-- CASTER WHEEL -->
@@ -73,4 +94,10 @@
                 <material name="black"/>
             </visual>
+            <collision>
+                <origin xyz="0.15 0 0.075" rpy="0 0 0" />
+                <geometry>
+                    <box size="0.3 0.3 0.15" />
+                </geometry>
+            </collision>
         </link>
 </robot>
