Commit message: fix bug collision

File: description/gazebo_control.xacro (robot description, xacro)
@@ -1,7 +1,7 @@
 <?xml version="1.0"?>
-<robot xmlns:xacro="http://www.ros.org/wiki/xacro" >
+<robot xmlns:xacro="http://www.ros.org/wiki/xacro" name="arap_bot">
     <gazebo>
         <plugin name='diff_drive' filename='libgazebo_ros_diff_drive.so'>
-            <!-- Joints -->
+            <!-- Wheel Information -->
             <left_joint>left_wheel_joint</left_joint>
             <right_joint>right_wheel_joint</right_joint>
@@ -9,19 +9,12 @@
             <wheel_diameter>0.1</wheel_diameter>
             <!-- Limits -->
-            <wheel_torque>10</wheel_torque>
-            <wheel_acceleration>2.0</wheel_acceleration>
-            <torque>5</torque>
-            <!-- topics  -->
-            <command_topic>cmd_vel</command_topic>
-            <odometry_topic>odom</odometry_topic>
-            <odometry_source>world</odometry_source>    <!-- odometrySource options "world" "encoder" -->
-            <!-- Frames -->
+            <max_wheel_torque>200</max_wheel_torque>
+            <max_wheel_acceleration>10.0</max_wheel_acceleration>
+            <!-- Output -->
             <odometry_frame>odom</odometry_frame>
             <robot_base_frame>base_link</robot_base_frame>
-            <!-- outputs -->
-            <publish_tf>1</publish_tf>
+            <publish_odom>true</publish_odom>
             <publish_odom_tf>true</publish_odom_tf>
             <publish_wheel_tf>true</publish_wheel_tf>
-            <publish_wheel_joint_state>true</publish_wheel_joint_state>
         </plugin>
     </gazebo>

File: description/robot.urdf.xacro (robot description, xacro)
@@ -2,5 +2,4 @@
 <robot xmlns:xacro="http://www.ros.org/wiki/xacro"  name="arap_bot">
     <xacro:include filename="gazebo_control.xacro" />
-    <xacro:include filename="inertial_macros.xacro" />
     <xacro:include filename="robot_core.xacro" />
 </robot>

File: description/robot_core.xacro (robot description, xacro)
@@ -1,24 +1,9 @@
-<?xml version="1.0" encoding="UTF-8"?>
-<robot xmlns:xacro="http://www.ros.org/wiki/xacro">
-    <material name="white">
-        <color rgba="1 1 1 1"/>
-    </material>
-    <material name="orange">
-        <color rgba="1 0.3 0.1 1"/>
-    </material>
-    <material name="blue">
-        <color rgba="0.2 0.2 1 1"/>
-    </material>
-    <material name="black">
-        <color rgba="0 0 0 1"/>
-    </material>
+<?xml version="1.0" ?>
+<robot xmlns:xacro="http://www.ros.org/wiki/xacro" name="arap_bot">
+    <xacro:include filename="inertial_macros.xacro" />
+    <xacro:include filename="colors.xacro" />
     <!-- BASE LINK-->
      <link name="base_link"></link>
      <!-- CHASSIS -->
-    <gazebo reference="chassis_link">
-        <material>Gazebo/White</material>
-        <mu1>0.001</mu1>
-        <mu2>0.001</mu2>
-    </gazebo>
     <link name="chassis_link" >
         <visual>
@@ -38,5 +23,5 @@
             <origin xyz="0.15 0 0.075" rpy="0 0 0"/>
         </xacro:inertial_box>
-  </link>
+    </link>
    <joint name="chassis_joint" type="fixed">
         <parent link="base_link" />
@@ -44,4 +29,7 @@
         <origin xyz="-0.1 0 0" />
    </joint>
+   <gazebo reference="chassis_link">
+        <material>Gazebo/White</material>
+    </gazebo>
    <!-- LEFT WHEEL-->
     <link name="left_wheel_link">
@@ -53,7 +41,6 @@
         </visual>
         <collision>
-            <origin xyz="0.15 0 0.075" rpy="0 0 0" />
             <geometry>
-                <box size="0.3 0.3 0.15" />
+                <cylinder length="0.04" radius="0.05" />
             </geometry>
         </collision>
@@ -85,4 +72,9 @@
             <material name="blue"/>
         </visual>
+        <collision>
+            <geometry>
+                <cylinder length="0.04" radius="0.05" />
+            </geometry>
+        </collision>
         <xacro:inertial_cylinder mass="0.1" length="0.05" radius="0.05">
             <origin xyz="0 0 0" rpy="0 0 0"/>
@@ -106,9 +98,13 @@
         </visual>
         <collision>
-            <origin xyz="0.15 0 0.075" rpy="0 0 0" />
             <geometry>
-                <box size="0.3 0.3 0.15" />
+                <sphere radius="0.05" />
             </geometry>
         </collision>
     </link>
+    <gazebo reference="caster_wheel_link">
+        <material>Gazebo/Black</material>
+        <mu1 value="0.001"/>
+        <mu2 value="0.001"/>
+    </gazebo>
 </robot>
