Commit message: complete core robot description

File: description/robot.urdf.xacro (robot description, xacro)
@@ -1,4 +1,5 @@
 <?xml version="1.0"?>
-<robot xmlns:xacro="http://www.ros.org/wiki/xacro"  name="robot">
+<robot xmlns:xacro="http://www.ros.org/wiki/xacro"  name="arap_bot">
+    <xacro:include filename="gazebo_control.xacro" />
     <xacro:include filename="inertial_macros.xacro" />
     <xacro:include filename="robot_core.xacro" />

File: description/robot_core.xacro (robot description, xacro)
@@ -16,88 +16,99 @@
      <link name="base_link"></link>
      <!-- CHASSIS -->
-      <link name="chassis_link" >
-            <visual>
-                <origin xyz="0.15 0 0.075" rpy="0 0 0" />
-                <geometry>
-                    <box size="0.3 0.3 0.15" />
-                </geometry>
-                <material name="white" />
-            </visual>
-            <collision>
-                <origin xyz="0.15 0 0.075" rpy="0 0 0" />
-                <geometry>
-                    <box size="0.3 0.3 0.15" />
-                </geometry>
-            </collision>
-            <xacro:inertial_box mass="0.5" x="0.3" y="0.3" z="0.15">
-                <origin xyz="0.15 0 0.075" rpy="0 0 0"/>
-            </xacro:inertial_box>
-      </link>
-       <joint name="chassis_joint" type="fixed">
-            <parent link="base_link" />
-            <child link="chassis_link" />
-            <origin xyz="-0.1 0 0" />
-       </joint>
-       <!-- LEFT WHEEL-->
-        <link name="left_wheel_link">
-            <visual>
-                <geometry>
-                    <cylinder length="0.04" radius="0.05" />
-                </geometry>
-                <material name="blue" />
-            </visual>
-            <collision>
-                <origin xyz="0.15 0 0.075" rpy="0 0 0" />
-                <geometry>
-                    <box size="0.3 0.3 0.15" />
-                </geometry>
-            </collision>
-            <xacro:inertial_cylinder mass="0.1" length="0.05" radius="0.05">
-                <origin xyz="0 0 0" rpy="0 0 0"/>
-            </xacro:inertial_cylinder>
-        </link>
-        <joint name="left_wheel_joint" type="continuous">
-            <parent link="base_link" />
-            <child link="left_wheel_link" />
-            <origin xyz="0 0.175 0" rpy="-${pi/2} 0 0" />
-            <axis xyz="0 0 1" />
-        </joint>
-        <!-- RIGHT WHEEL -->
-        <joint name="right_wheel_joint" type="continuous">
-            <parent link="base_link"/>
-            <child link="right_wheel"/>
-            <origin xyz="0 -0.175 0" rpy="${pi/2} 0 0"/>
-            <axis xyz="0 0 -1"/>
-        </joint>
-        <link name="right_wheel">
-            <visual>joint_state_publisher_gui
-                <geometry>
-                    <cylinder length="0.04" radius="0.05" />
-                </geometry>
-                <material name="blue"/>
-            </visual>
-            <xacro:inertial_sphere mass="0.1" radius="0.05">
-                <origin xyz="0 0 0" rpy="0 0 0"/>
-            </xacro:inertial_sphere>
-        </link>
-        <!-- CASTER WHEEL -->
-        <joint name="caster_wheel_joint" type="fixed">
-            <parent link="chassis_link"/>
-            <child link="caster_wheel"/>
-            <origin xyz="0.24 0 0" rpy="0 0 0"/>
-        </joint>
-        <link name="caster_wheel">
-            <visual>
-                <geometry>
-                    <sphere radius="0.05" />
-                </geometry>
-                <material name="black"/>
-            </visual>
-            <collision>
-                <origin xyz="0.15 0 0.075" rpy="0 0 0" />
-                <geometry>
-                    <box size="0.3 0.3 0.15" />
-                </geometry>
-            </collision>
-        </link>
+    <gazebo reference="chassis_link">
+        <material>Gazebo/White</material>
+        <mu1>0.001</mu1>
+        <mu2>0.001</mu2>
+    </gazebo>
+    <link name="chassis_link" >
+        <visual>
+            <origin xyz="0.15 0 0.075" rpy="0 0 0" />
+            <geometry>
+                <box size="0.3 0.3 0.15" />
+            </geometry>
+            <material name="white" />
+        </visual>
+        <collision>
+            <origin xyz="0.15 0 0.075" rpy="0 0 0" />
+            <geometry>
+                <box size="0.3 0.3 0.15" />
+            </geometry>
+        </collision>
+        <xacro:inertial_box mass="0.5" x="0.3" y="0.3" z="0.15">
+            <origin xyz="0.15 0 0.075" rpy="0 0 0"/>
+        </xacro:inertial_box>
+  </link>
+   <joint name="chassis_joint" type="fixed">
+        <parent link="base_link" />
+        <child link="chassis_link" />
+        <origin xyz="-0.1 0 0" />
+   </joint>
+   <!-- LEFT WHEEL-->
+    <link name="left_wheel_link">
+        <visual>
+            <geometry>
+                <cylinder length="0.04" radius="0.05" />
+            </geometry>
+            <material name="blue" />
+        </visual>
+        <collision>
+            <origin xyz="0.15 0 0.075" rpy="0 0 0" />
+            <geometry>
+                <box size="0.3 0.3 0.15" />
+            </geometry>
+        </collision>
+        <xacro:inertial_cylinder mass="0.1" length="0.05" radius="0.05">
+            <origin xyz="0 0 0" rpy="0 0 0"/>
+        </xacro:inertial_cylinder>
+    </link>
+    <joint name="left_wheel_joint" type="continuous">
+        <parent link="base_link" />
+        <child link="left_wheel_link" />
+        <origin xyz="0 0.175 0" rpy="-${pi/2} 0 0" />
+        <axis xyz="0 0 1" />
+    </joint>
+    <gazebo reference="left_wheel_link">
+        <material>Gazebo/Blue</material>
+    </gazebo>
+    <!-- RIGHT WHEEL -->
+    <joint name="right_wheel_joint" type="continuous">
+        <parent link="base_link"/>
+        <child link="right_wheel_link"/>
+        <origin xyz="0 -0.175 0" rpy="${pi/2} 0 0"/>
+        <axis xyz="0 0 -1"/>
+    </joint>
+    <link name="right_wheel_link">
+        <visual>
+            <geometry>
+                <cylinder length="0.04" radius="0.05" />
+            </geometry>
+            <material name="blue"/>
+        </visual>
+        <xacro:inertial_cylinder mass="0.1" length="0.05" radius="0.05">
+            <origin xyz="0 0 0" rpy="0 0 0"/>
+        </xacro:inertial_cylinder>
+    </link>
+    <gazebo reference="right_wheel_link">
+        <material>Gazebo/Blue</material>
+    </gazebo>
+    <!-- CASTER WHEEL -->
+    <joint name="caster_wheel_joint" type="fixed">
+        <parent link="chassis_link"/>
+        <child link="caster_wheel_link"/>
+        <origin xyz="0.24 0 0" rpy="0 0 0"/>
+    </joint>
+    <link name="caster_wheel_link">
+        <visual>
+            <geometry>
+                <sphere radius="0.05" />
+            </geometry>
+            <material name="black"/>
+        </visual>
+        <collision>
+            <origin xyz="0.15 0 0.075" rpy="0 0 0" />
+            <geometry>
+                <box size="0.3 0.3 0.15" />
+            </geometry>
+        </collision>
+    </link>
 </robot>

Commit message: refactor

File: description/robot.urdf.xacro (robot description, xacro)
@@ -1,5 +1,8 @@
 <?xml version="1.0"?>
 <robot xmlns:xacro="http://www.ros.org/wiki/xacro"  name="arap_bot">
+    <xacro:include filename="inertial_macros.xacro" />
+    <xacro:include filename="colors.xacro" />
     <xacro:include filename="gazebo_control.xacro" />
+    <xacro:include filename="lidar.xacro" />
     <xacro:include filename="robot_core.xacro" />
 </robot>

File: description/robot_core.xacro (robot description, xacro)
@@ -1,6 +1,4 @@
 <?xml version="1.0" ?>
 <robot xmlns:xacro="http://www.ros.org/wiki/xacro" name="arap_bot">
-    <xacro:include filename="inertial_macros.xacro" />
-    <xacro:include filename="colors.xacro" />
     <!-- BASE LINK-->
      <link name="base_link"></link>
@@ -24,10 +22,10 @@
         </xacro:inertial_box>
     </link>
-   <joint name="chassis_joint" type="fixed">
+    <joint name="chassis_joint" type="fixed">
         <parent link="base_link" />
         <child link="chassis_link" />
         <origin xyz="-0.1 0 0" />
-   </joint>
-   <gazebo reference="chassis_link">
+    </joint>
+    <gazebo reference="chassis_link">
         <material>Gazebo/White</material>
     </gazebo>
